Commit message: add the stl files

File: description/robot_core.xacro (robot description, xacro)
@@ -263,3 +263,8 @@
     <joint_properties friction="0.0"/>
   </joint>
+  <joint name="dummy_joint" type="fixed">
+    <parent link="dummy_link"/>
+    <child link="corps"/>
+    <origin xyz="0 0 0"/>
+  </joint>
 </robot>

Commit message: add the stl files

File: description/robot_core.xacro (robot description, xacro)
@@ -5,5 +5,5 @@
       <origin xyz="-0.16487494494899462838 0.00098504563636114816916 -0.036950519133039851083" rpy="0 -0 0" />
       <geometry>
-        <mesh filename="package:///corps.stl"/>
+        <mesh filename="package://my_bot/cadstl/corps.stl"/>
       </geometry>
       <material name="corps_material">
@@ -14,5 +14,5 @@
       <origin xyz="-0.16487494494899462838 0.00098504563636114816916 -0.036950519133039851083" rpy="0 -0 0" />
       <geometry>
-        <mesh filename="package:///corps.stl"/>
+        <mesh filename="package://my_bot/cadstl/corps.stl"/>
       </geometry>
     </collision>
@@ -27,5 +27,5 @@
       <origin xyz="0 0 0.035801747109368328714" rpy="3.141592653589793116 -0 1.0379658610783623998e-17" />
       <geometry>
-        <mesh filename="package:///support_roue.stl"/>
+        <mesh filename="package://my_bot/cadstl/support_roue.stl"/>
       </geometry>
       <material name="support_roue_material">
@@ -36,5 +36,5 @@
       <origin xyz="0 0 0.035801747109368328714" rpy="3.141592653589793116 -0 1.0379658610783623998e-17" />
       <geometry>
-        <mesh filename="package:///support_roue.stl"/>
+        <mesh filename="package://my_bot/cadstl/support_roue.stl"/>
       </geometry>
     </collision>
@@ -49,5 +49,5 @@
       <origin xyz="0 0 0.017999999999999960476" rpy="3.141592653589793116 8.1540335100360869226e-18 0" />
       <geometry>
-        <mesh filename="package:///roue.stl"/>
+        <mesh filename="package://my_bot/cadstl/roue.stl"/>
       </geometry>
       <material name="roue_material">
@@ -58,5 +58,5 @@
       <origin xyz="0 0 0.017999999999999960476" rpy="3.141592653589793116 8.1540335100360869226e-18 0" />
       <geometry>
-        <mesh filename="package:///roue.stl"/>
+        <mesh filename="package://my_bot/cadstl/roue.stl"/>
       </geometry>
     </collision>
@@ -87,5 +87,5 @@
       <origin xyz="0 -2.7755575615628913511e-17 0.035801747109368328714" rpy="3.141592653589793116 -0 1.8377189892559446398e-18" />
       <geometry>
-        <mesh filename="package:///support_roue.stl"/>
+        <mesh filename="package://my_bot/cadstl/support_roue.stl"/>
       </geometry>
       <material name="support_roue_material">
@@ -96,5 +96,5 @@
       <origin xyz="0 -2.7755575615628913511e-17 0.035801747109368328714" rpy="3.141592653589793116 -0 1.8377189892559446398e-18" />
       <geometry>
-        <mesh filename="package:///support_roue.stl"/>
+        <mesh filename="package://my_bot/cadstl/support_roue.stl"/>
       </geometry>
     </collision>
@@ -109,5 +109,5 @@
       <origin xyz="0 0 -0.018000000000000015987" rpy="2.5242800315414714867e-18 -4.1786896273659949387e-19 -5.5878178144470137785e-18" />
       <geometry>
-        <mesh filename="package:///roue.stl"/>
+        <mesh filename="package://my_bot/cadstl/roue.stl"/>
       </geometry>
       <material name="roue_material">
@@ -118,5 +118,5 @@
       <origin xyz="0 0 -0.018000000000000015987" rpy="2.5242800315414714867e-18 -4.1786896273659949387e-19 -5.5878178144470137785e-18" />
       <geometry>
-        <mesh filename="package:///roue.stl"/>
+        <mesh filename="package://my_bot/cadstl/roue.stl"/>
       </geometry>
     </collision>
@@ -147,5 +147,5 @@
       <origin xyz="0 0 0.035801747109368328714" rpy="3.141592653589793116 -0 3.985001973689215218e-19" />
       <geometry>
-        <mesh filename="package:///support_roue.stl"/>
+        <mesh filename="package://my_bot/cadstl/support_roue.stl"/>
       </geometry>
       <material name="support_roue_material">
@@ -156,5 +156,5 @@
       <origin xyz="0 0 0.035801747109368328714" rpy="3.141592653589793116 -0 3.985001973689215218e-19" />
       <geometry>
-        <mesh filename="package:///support_roue.stl"/>
+        <mesh filename="package://my_bot/cadstl/support_roue.stl"/>
       </geometry>
     </collision>
@@ -169,5 +169,5 @@
       <origin xyz="0 1.3877787807814456755e-17 0.018000000000000002109" rpy="-3.141592653589793116 2.6771850920217469288e-18 3.0984265678640010969e-17" />
       <geometry>
-        <mesh filename="package:///roue.stl"/>
+        <mesh filename="package://my_bot/cadstl/roue.stl"/>
       </geometry>
       <material name="roue_material">
@@ -178,5 +178,5 @@
       <origin xyz="0 1.3877787807814456755e-17 0.018000000000000002109" rpy="-3.141592653589793116 2.6771850920217469288e-18 3.0984265678640010969e-17" />
       <geometry>
-        <mesh filename="package:///roue.stl"/>
+        <mesh filename="package://my_bot/cadstl/roue.stl"/>
      </geometry>
     </collision>
@@ -207,5 +207,5 @@
       <origin xyz="0 1.3877787807814456755e-17 0.035801747109368328714" rpy="3.141592653589793116 -0 8.6963759104196122014e-18" />
       <geometry>
-        <mesh filename="package:///support_roue.stl"/>
+        <mesh filename="package://my_bot/cadstl/support_roue.stl"/>
       </geometry>
       <material name="support_roue_material">
@@ -216,5 +216,5 @@
       <origin xyz="0 1.3877787807814456755e-17 0.035801747109368328714" rpy="3.141592653589793116 -0 8.6963759104196122014e-18" />
       <geometry>
-        <mesh filename="package:///support_roue.stl"/>
+        <mesh filename="package://my_bot/cadstl/support_roue.stl"/>
       </geometry>
     </collision>
@@ -229,5 +229,5 @@
       <origin xyz="0 0 0.018000000000000015987" rpy="3.141592653589793116 -2.8063591805892701907e-20 3.8063495312512622149e-19" />
       <geometry>
-        <mesh filename="package:///roue.stl"/>
+        <mesh filename="package://my_bot/cadstl/roue.stl"/>
       </geometry>
       <material name="roue_material">
@@ -238,5 +238,5 @@
       <origin xyz="0 0 0.018000000000000015987" rpy="3.141592653589793116 -2.8063591805892701907e-20 3.8063495312512622149e-19" />
       <geometry>
-        <mesh filename="package:///roue.stl"/>
+        <mesh filename="package://my_bot/cadstl/roue.stl"/>
       </geometry>
     </collision>
@@ -263,4 +263,11 @@
     <joint_properties friction="0.0"/>
   </joint>
+  <link name="dummy_link">
+    <inertial>
+      <mass value="0.0001"/> <!-- A very small mass to avoid numerical instability -->
+      <origin xyz="0 0 0"/>
+      <inertia ixx="0.0001" ixy="0" ixz="0" iyy="0.0001" iyz="0" izz="0.0001"/>
+    </inertial>
+  </link>
   <joint name="dummy_joint" type="fixed">
     <parent link="dummy_link"/>

Commit message: file instead of package

File: description/robot_core.xacro (robot description, xacro)
@@ -5,5 +5,5 @@
       <origin xyz="-0.16487494494899462838 0.00098504563636114816916 -0.036950519133039851083" rpy="0 -0 0" />
       <geometry>
-        <mesh filename="package://my_bot/cadstl/corps.stl"/>
+        <mesh filename="file://cadstl/corps.stl"/>
       </geometry>
       <material name="corps_material">
@@ -14,5 +14,5 @@
       <origin xyz="-0.16487494494899462838 0.00098504563636114816916 -0.036950519133039851083" rpy="0 -0 0" />
       <geometry>
-        <mesh filename="package://my_bot/cadstl/corps.stl"/>
+        <mesh filename="file://cadstl/corps.stl"/>
       </geometry>
     </collision>
@@ -27,5 +27,5 @@
       <origin xyz="0 0 0.035801747109368328714" rpy="3.141592653589793116 -0 1.0379658610783623998e-17" />
       <geometry>
-        <mesh filename="package://my_bot/cadstl/support_roue.stl"/>
+        <mesh filename="file://cadstl/support_roue.stl"/>
       </geometry>
       <material name="support_roue_material">
@@ -36,5 +36,5 @@
       <origin xyz="0 0 0.035801747109368328714" rpy="3.141592653589793116 -0 1.0379658610783623998e-17" />
       <geometry>
-        <mesh filename="package://my_bot/cadstl/support_roue.stl"/>
+        <mesh filename="file://cadstl/support_roue.stl"/>
       </geometry>
     </collision>
@@ -49,5 +49,5 @@
       <origin xyz="0 0 0.017999999999999960476" rpy="3.141592653589793116 8.1540335100360869226e-18 0" />
       <geometry>
-        <mesh filename="package://my_bot/cadstl/roue.stl"/>
+        <mesh filename="file://cadstl/roue.stl"/>
       </geometry>
       <material name="roue_material">
@@ -58,5 +58,5 @@
       <origin xyz="0 0 0.017999999999999960476" rpy="3.141592653589793116 8.1540335100360869226e-18 0" />
       <geometry>
-        <mesh filename="package://my_bot/cadstl/roue.stl"/>
+        <mesh filename="file://cadstl/roue.stl"/>
       </geometry>
     </collision>
@@ -87,5 +87,5 @@
       <origin xyz="0 -2.7755575615628913511e-17 0.035801747109368328714" rpy="3.141592653589793116 -0 1.8377189892559446398e-18" />
       <geometry>
-        <mesh filename="package://my_bot/cadstl/support_roue.stl"/>
+        <mesh filename="file://cadstl/support_roue.stl"/>
       </geometry>
       <material name="support_roue_material">
@@ -96,5 +96,5 @@
       <origin xyz="0 -2.7755575615628913511e-17 0.035801747109368328714" rpy="3.141592653589793116 -0 1.8377189892559446398e-18" />
       <geometry>
-        <mesh filename="package://my_bot/cadstl/support_roue.stl"/>
+        <mesh filename="file://cadstl/support_roue.stl"/>
       </geometry>
     </collision>
@@ -109,5 +109,5 @@
       <origin xyz="0 0 -0.018000000000000015987" rpy="2.5242800315414714867e-18 -4.1786896273659949387e-19 -5.5878178144470137785e-18" />
       <geometry>
-        <mesh filename="package://my_bot/cadstl/roue.stl"/>
+        <mesh filename="file://cadstl/roue.stl"/>
       </geometry>
       <material name="roue_material">
@@ -118,5 +118,5 @@
       <origin xyz="0 0 -0.018000000000000015987" rpy="2.5242800315414714867e-18 -4.1786896273659949387e-19 -5.5878178144470137785e-18" />
       <geometry>
-        <mesh filename="package://my_bot/cadstl/roue.stl"/>
+        <mesh filename="file://cadstl/roue.stl"/>
       </geometry>
     </collision>
@@ -147,5 +147,5 @@
       <origin xyz="0 0 0.035801747109368328714" rpy="3.141592653589793116 -0 3.985001973689215218e-19" />
       <geometry>
-        <mesh filename="package://my_bot/cadstl/support_roue.stl"/>
+        <mesh filename="file://cadstl/support_roue.stl"/>
       </geometry>
       <material name="support_roue_material">
@@ -156,5 +156,5 @@
       <origin xyz="0 0 0.035801747109368328714" rpy="3.141592653589793116 -0 3.985001973689215218e-19" />
       <geometry>
-        <mesh filename="package://my_bot/cadstl/support_roue.stl"/>
+        <mesh filename="file://cadstl/support_roue.stl"/>
       </geometry>
     </collision>
@@ -169,5 +169,5 @@
       <origin xyz="0 1.3877787807814456755e-17 0.018000000000000002109" rpy="-3.141592653589793116 2.6771850920217469288e-18 3.0984265678640010969e-17" />
       <geometry>
-        <mesh filename="package://my_bot/cadstl/roue.stl"/>
+        <mesh filename="file://cadstl/roue.stl"/>
       </geometry>
       <material name="roue_material">
@@ -178,5 +178,5 @@
       <origin xyz="0 1.3877787807814456755e-17 0.018000000000000002109" rpy="-3.141592653589793116 2.6771850920217469288e-18 3.0984265678640010969e-17" />
       <geometry>
-        <mesh filename="package://my_bot/cadstl/roue.stl"/>
+        <mesh filename="file://cadstl/roue.stl"/>
      </geometry>
     </collision>
@@ -207,5 +207,5 @@
       <origin xyz="0 1.3877787807814456755e-17 0.035801747109368328714" rpy="3.141592653589793116 -0 8.6963759104196122014e-18" />
       <geometry>
-        <mesh filename="package://my_bot/cadstl/support_roue.stl"/>
+        <mesh filename="file://cadstl/support_roue.stl"/>
       </geometry>
       <material name="support_roue_material">
@@ -216,5 +216,5 @@
       <origin xyz="0 1.3877787807814456755e-17 0.035801747109368328714" rpy="3.141592653589793116 -0 8.6963759104196122014e-18" />
       <geometry>
-        <mesh filename="package://my_bot/cadstl/support_roue.stl"/>
+        <mesh filename="file://cadstl/support_roue.stl"/>
       </geometry>
     </collision>
@@ -229,5 +229,5 @@
       <origin xyz="0 0 0.018000000000000015987" rpy="3.141592653589793116 -2.8063591805892701907e-20 3.8063495312512622149e-19" />
       <geometry>
-        <mesh filename="package://my_bot/cadstl/roue.stl"/>
+        <mesh filename="file://cadstl/roue.stl"/>
       </geometry>
       <material name="roue_material">
@@ -238,5 +238,5 @@
       <origin xyz="0 0 0.018000000000000015987" rpy="3.141592653589793116 -2.8063591805892701907e-20 3.8063495312512622149e-19" />
       <geometry>
-        <mesh filename="package://my_bot/cadstl/roue.stl"/>
+        <mesh filename="file://cadstl/roue.stl"/>
       </geometry>
     </collision>
